File: hardware/power_distribution/power_distribution.sch (EAGLE design)
At the start: 29 parts, among them Q1 MOSFET-NCHANNELFQP30N06L, Q2 MOSFET-NCHANNELFQP30N06L, U1 LTC4412ES6PBF, U10 ATMEGA328P_PDIP, U2 LTC4412ES6PBF, U3 ACS712, U4 ACS712, U5 MAX233, U6 MAX233, X1 53048-04, X4 53048-04, X5 53048-04, Y1 16MHz

Commit message: Balances battery voltages and outputs one combined voltage
Parts:
- removed F1, F2: FUSE-HOLDER, fuse-holder:FUSE-HOLDER
- removed JP1: CARD_EDGE, Molex_Edge_2:CARD_EDGE
- removed R1, R2: 10k, resistor:R-TRIMM43P
- removed U1, U2: LTC4412ES6PBF, LTC_By_element14_Batch_1:LTC4412ES6PBF
- removed U10: ATMEGA328P_PDIP, SparkFun-DigitalIC:ATMEGA328P_PDIP
- removed U3, U4: ACS712, SparkFun-AnalogIC:ACS712
- removed U5, U6: MAX233, maxim:MAX233
- removed X1, X4, X5: 53048-04, con-molex:53048-04
- removed Y1: 16MHz, crystal:CRYSTALHC49U-V
- added 5V, 5V_GND, BALANCED+, BALANCED_GND, GATE1, GATE1_GND, GATE2, GATE2_GND, RAW_V1, RAW_V1_GND, RAW_V2, RAW_V2_GND, SCL, SCL_GND, SDA, SDA_GND: TPPAD1-13, testpad:TPPAD1-13
- added C10: 0.1uF, SparkFun-Capacitors:0.1UF-KIT-EZ-50V-20%
- added CURRENT1, CURRENT2, RAW, VOLTAGE1, VOLTAGE2: (no value), led:LED3MM
- added CURRENT_SENSOR1, CURRENT_SENSOR2: ACS712ELCTR-05B-T, Allegro_By_element14_Batch_1:ACS712ELCTR-05B-T
- added INPUT1, INPUT2, OUTPUT: MOLEX172043-0201, Molex172043-0201:MOLEX172043-0201
- added ISP1: AVRISP-6, adafruit:AVRISP-6
- added MICROCONTROLLER: ATMEGA168P-20PU, Atmel_By_element14_Batch_1-00:ATMEGA168P-20PU
- added Q3: 60V/32A/35mΩ, SparkFun-DiscreteSemi:MOSFET-NCH-FQP30N06L
- added R3, R4, R5, R6, R7: (no value), resistor:R-US_0207/12
- added SW1: (no value), adafruit:SWITCH_PUSHBUTTONEVQ-PE
- added U$3: 1-530844-7, 1-530844-7-PCBEDGE:1-530844-7
- added U$4, U$5: ADM1293, Analog Devices_By_element14_Batch_1:ADM1293
- added V_BALANCER1, V_BALANCER_2: LTC4352CDDPBF, LTC_By_element14_Batch_1:LTC4352CDDPBF
- C1, C2, C3: device SparkFun-Capacitors:CAPEZ -> SparkFun-Capacitors:0.1UF-KIT-EZ-50V-20%
- C4: value (none) -> 0.1uF; device SparkFun-Capacitors:CAPEZ -> SparkFun-Capacitors:0.1UF-KIT-EZ-50V-20%
- C5: value 0.1uF -> 20pF; device SparkFun-Capacitors:CAPEZ -> SparkFun-Capacitors:0.1UF-KIT-EZ-50V-20%
- C6: value 1.0uF -> 20pF; device SparkFun-Capacitors:CAPEZ -> SparkFun-Capacitors:0.1UF-KIT-EZ-50V-20%
- C7: value 1.0uF -> 0.1uF; device SparkFun-Capacitors:CAPEZ -> SparkFun-Capacitors:0.1UF-KIT-EZ-50V-20%
- C8, C9: value 20pF -> 0.1uF; device SparkFun-Capacitors:CAPEZ -> SparkFun-Capacitors:0.1UF-KIT-EZ-50V-20%
- Q1: value MOSFET-NCHANNELFQP30N06L -> (none); device SparkFun-DiscreteSemi:MOSFET-NCHANNELFQP30N06L -> crystal:CRYSTALHC49U-V
- Q2: value MOSFET-NCHANNELFQP30N06L -> 60V/32A/35mΩ; device SparkFun-DiscreteSemi:MOSFET-NCHANNELFQP30N06L -> SparkFun-DiscreteSemi:MOSFET-NCH-FQP30N06L
- U$1, U$2: value MOLEX172043-0201 -> C1H30; device Molex172043-0201:MOLEX172043-0201 -> fuse:C1H30
Connections:
- removed net B+: C4.1, JP1.B+, Q1.D, Q2.D, U1.SENSE, U2.SENSE
- removed net B-: C4.2, JP1.B-, U$1.PIN2, U$2.PIN2
- removed net B1+: F1.P$1, U$1.PIN1
- removed net B1F+: F1.P$2, R1.A, U3.IP+@1, U3.IP+@2
- removed net B1RX232: U5G$1.R1IN, X4-3.S
- removed net B1TX232: U5G$1.T1OUT, X4-2.S
- removed net B2+: F2.P$1, U$2.PIN1
- removed net B2F+: F2.P$2, R2.A, U4.IP+@1, U4.IP+@2
- removed net B2RX232: U5G$1.R2IN, X5-3.S
- removed net B2TX232: U5G$1.T2OUT, X5-2.S
- removed net C2+B: U5G$1.C2+@1, U5G$1.C2+@2
- removed net C2+CPU: U6G$1.C2+@1, U6G$1.C2+@2
- removed net C2-B: U5G$1.C2-@1, U5G$1.C2-@2
- removed net C2-CPU: U6G$1.C2-@1, U6G$1.C2-@2
- removed net CPU232RX: U6G$1.R1IN, X1-3.S
- removed net CPU232TX: U6G$1.T1OUT, X1-2.S
- removed net FILT1: C2.1, U3.FILT
- removed net FILT2: C1.1, U4.FILT
- removed net RX1SOFT: U10.PD5(T1), U5G$1.R1OUT
- removed net RX2SOFT: U10.PB1(OC1A), U5G$1.R2OUT
- removed net RXD: U10.PD0(RXD), U6G$1.R1OUT
- removed net TX1SOFT: U10.PD6(AIN0), U5G$1.T1IN
- removed net TX2SOFT: U10.PB2(SS/OC1B), U5G$1.T2IN
- removed net TXD: U10.PD1(TXD), U6G$1.T1IN
- removed net V-B: U5G$1.V-@1, U5G$1.V-@2
- removed net V-CPU: U6G$1.V-@1, U6G$1.V-@2
- removed net VDIV1: R1.S, U10.PC1(ADC1)
- removed net VDIV2: R2.S, U10.PC2(ADC2)
- removed net VIN1: Q1.S, U1.VIN, U3.IP-@3, U3.IP-@4
- removed net VIN2: Q2.S, U2.VIN, U4.IP-@3, U4.IP-@4
- removed net VOUT1: U10.PC0(ADC0), U3.VOUT
- removed net VOUT2: U10.PC3(ADC3), U4.VOUT
- removed net XOSC1: C8.2, U10.PB6(XTAL1/TOSC1), Y1.1
- removed net XOSC2: C9.2, U10.PB7(XTAL2/TOSC2), Y1.2
- new net CURRENT_LED1: MICROCONTROLLER.PD0, R4.1
- new net CURRENT_LED2: MICROCONTROLLER.PD1, R5.1
- new net CURRENT_SIG1: CURRENT_SENSOR1.VIOUT, MICROCONTROLLER.PC0
- new net CURRENT_SIG2: CURRENT_SENSOR2.VIOUT, MICROCONTROLLER.PC2
- new net MISO: ISP1.MISO, MICROCONTROLLER.PB4
- new net MOSI: ISP1.MOSI, MICROCONTROLLER.PB3
- new net N$1: C9.1, CURRENT_SENSOR1.IP+, CURRENT_SENSOR1.IP+_2, U$1.2, U$4.VCC, U$4.VIN
- new net N$10: INPUT1.RAW+, RAW_V1.TP, U$1.1
- new net N$11: C10.1, CURRENT_SENSOR2.IP+, CURRENT_SENSOR2.IP+_2, U$2.2, U$5.VCC, U$5.VIN
- new net N$13: CURRENT2.A, R5.2
- new net N$14: C2.1, CURRENT_SENSOR1.FILTER
- new net N$15: R6.2, VOLTAGE1.A
- new net N$16: INPUT2.RAW+, RAW_V2.TP, U$2.1
- new net N$17: R7.2, VOLTAGE2.A
- new net N$18: C4.1, CURRENT_SENSOR2.FILTER
- new net N$19: BALANCED_GND.TP, C10.2, C9.2, INPUT1.RAW-, INPUT2.RAW-, OUTPUT.RAW-, RAW.C, RAW_V1_GND.TP, RAW_V2_GND.TP, U$4.ADR1, U$4.ADR2, U$4.GND, U$5.GND
- new net N$2: C5.1, MICROCONTROLLER.PB6, Q1.1
- new net N$26: BALANCED+.TP, OUTPUT.RAW+, Q2.D, Q3.D, R3.1, V_BALANCER1.OUT, V_BALANCER_2.OUT
- new net N$27: MICROCONTROLLER.PC6, SW1.P$2
- new net N$3: C7.1, V_BALANCER_2.UV, V_BALANCER_2.VCC
- new net N$4: C6.1, Q1.2
- new net N$5: CURRENT_SENSOR1.IP-, CURRENT_SENSOR1.IP-_2, Q3.S, V_BALANCER1.VIN
- new net N$7: CURRENT1.A, R4.2
- new net N$8: R3.2, RAW.A
- new net N$9: C8.1, V_BALANCER1.UV, V_BALANCER1.VCC
- new net RESET_SW: ISP1.RST, SW1.P$1
- new net SCK: ISP1.SCK, MICROCONTROLLER.PB5
- new net VOLTAGE_IN2: CURRENT_SENSOR2.IP-, CURRENT_SENSOR2.IP-_2, Q2.S, V_BALANCER_2.VIN
- new net VOLTAGE_LED1: MICROCONTROLLER.PD2, R6.1
- new net VOLTAGE_LED2: MICROCONTROLLER.PD3, R7.1
- net GATE1: now also GATE1.TP, Q3.G, V_BALANCER1.GATE; no longer Q1.G, U1.GATE
- net GATE2: now also GATE2.TP, V_BALANCER_2.GATE; no longer U2.GATE
- net GND: now also 5V_GND.TP, C4.2, C8.2, CURRENT1.C, CURRENT2.C, CURRENT_SENSOR1.GND, CURRENT_SENSOR2.GND, GATE1_GND.TP, GATE2_GND.TP, ISP1.GND, MICROCONTROLLER.GND, MICROCONTROLLER.GND_2, SCL_GND.TP, SDA_GND.TP, U$3.5V_GND_P1, U$3.5V_GND_P2, U$3.5V_GND_P3, U$3.5V_GND_P4, U$3.5V_GND_P5, U$3.5V_GND_P6, VOLTAGE1.C, VOLTAGE2.C, V_BALANCER1.GND, V_BALANCER1.OV, V_BALANCER1.REV, V_BALANCER_2.GND, V_BALANCER_2.OV, V_BALANCER_2.REV; no longer C8.1, C9.1, JP1.GND, R1.E, R2.E, U1.CTL, U1.GND, U10.GND@1, U10.GND@2, U2.CTL, U2.GND, U3.GND, U4.GND, U5P.GND@1, U5P.GND@2, U6P.GND@1, U6P.GND@2, X1-4.S, X4-4.S, X5-4.S
- net SCL: now also MICROCONTROLLER.PC5, SCL.TP, U$3.SCL_SENSOR, U$4.SCL, U$5.SCL; no longer JP1.12VS, U10.PC5(ADC5/SCL)
- net SDA: now also MICROCONTROLLER.PC4, SDA.TP, U$3.SDA_SENSOR, U$4.SDAI, U$4.SDAO, U$5.SDAI, U$5.SDAO; no longer JP1.5VS_KILL, U10.PC4(ADC4/SDA)
- net VCC: now also 5V.TP, C1.1, CURRENT_SENSOR1.VCC, CURRENT_SENSOR2.VCC, ISP1.VCC, MICROCONTROLLER.AREF, MICROCONTROLLER.AVCC, MICROCONTROLLER.VCC, U$3.5V_P1, U$3.5V_P2, U$3.5V_P3, U$3.5V_P4, U$3.5V_P5, U$3.5V_P6; no longer C5.1, C6.1, C7.1, JP1.5V, U10.AREF, U10.AVCC, U10.VCC, U3.VCC, U4.VCC, U5P.VCC, U6P.VCC, X4-1.S, X5-1.S
Other:
- note added: "ADM1293-1BARUZ"
- note added: "Address: (Binary) 0110000X (Hex) 0x30"
- note added: "Address: (Binary) 0111010X (Hex) 0x3A"
- note added: "Balanced Battery Voltage 1"
- note added: "Balanced Battery Voltage 2"
- note added: "Balanced Voltage Output"
- note added: "Battery Input 1"
- note added: "Battery Input 2"
- note added: "ISP Header"
- note added: "Voltage Monitor"
- moved on the sheet: C1, C2, C3, C4, C5, C6, C7, C8, C9
